File: ai03-pcb-guide/_autosave-ai03-pcb-guide.kicad_pcb (KiCad board)
At the start: 2 copper layers, 77 x 38.1 mm, 24 parts, among them SW1 SW_Push, U1 ATmega32U4-A, Y1 Crystal_GND24_Small

Commit message: finishing up pcb
Parts:
- MX1, MX2, MX3, MX4: footprint MX_Alps_Hybrid:MX-1U-NoLED -> MX_Alps_Hybrid:MX-1U
Routing:
- net Net-(D3-Pad2): track 7.38 -> 4.11 mm
- net Net-(D2-Pad2): track 8.81 -> 5.97 mm
- net Net-(D4-Pad2): track 8.48 -> 6.49 mm
- net Net-(D1-Pad2): track 7.49 -> 5.81 mm
- net ROW1: track 55.0 -> 54.3 mm
- net ROW0: track 46.7 -> 47.4 mm
