File: ai03-pcb-guide/ai03-pcb-guide.sch (KiCad schematic (older format))
At the start: 14 parts

Commit message: Please enter the commit message for your changes. Lines starting
Finishing schematic
Parts:
- added D1, D2, D3, D4: D_Small, symbol Device:D_Small
- added F1: 500mA, symbol Device:Polyfuse
- added MX1, MX2, MX3, MX4: MX-NoLED, symbol MX_Alps_Hybrid:MX-NoLED
- added USB1: Molex-0548190589, symbol random-keyboard-parts:Molex-0548190589
- C1, C2, C3, C4, C5, C6, C7: renamed from C?; footprint (none) -> Capacitor_SMD:C_0805_2012Metric
- gave numbers to parts that had none: 7
Connections:
- net +5V: now also F1.1
- net D+: now also USB1.3 (D+)
- net D-: now also USB1.4 (D-)
- net GND: now also USB1.1 (GND)
- new net: D1.2 (A), MX1.2 (ROW)
- new net: D2.2 (A), MX2.2 (ROW)
- new net: D3.2 (A), MX3.2 (ROW)
- new net: D4.2 (A), MX4.2 (ROW)
- new net COL0: MX1.1 (COL), MX3.1 (COL)
- new net COL1: MX2.1 (COL), MX4.1 (COL)
- new net ROW0: D1.1 (K), D2.1 (K)
- new net ROW1: D3.1 (K), D4.1 (K)
- new net VCC: F1.2, USB1.5 (VBUS)

Commit message: finishing schematic
Parts:
- D1, D2, D3, D4: footprint (none) -> Diode_SMD:D_SOD-123
- F1: footprint (none) -> Fuse:Fuse_1206_3216Metric
- MX1, MX2, MX3, MX4: footprint (none) -> MX_Alps_Hybrid:MX-1U-NoLED
- R1, R2, R3, R4: footprint (none) -> Resistor_SMD:R_0805_2012Metric
- SW1: footprint (none) -> random-keyboard-parts:SKQG-1155865
- USB1: footprint (none) -> random-keyboard-parts:Molex-0548190589
- Y1: footprint (none) -> Crystal:Crystal_SMD_3225-4Pin_3.2x2.5mm
Changed lines of the file:
@@
 F 0 "R4" V 10104 3600 50  0000 C CNN
 F 1 "10k" V 10195 3600 50  0000 C CNN
-F 2 "" H 10300 3600 50  0001 C CNN
+F 2 "Resistor_SMD:R_0805_2012Metric" H 10300 3600 50  0001 C CNN
 F 3 "~" H 10300 3600 50  0001 C CNN
 	1    10300 3600
@@
 F 0 "R3" V 7293 2600 50  0000 C CNN
 F 1 "22" V 7384 2600 50  0000 C CNN
-F 2 "" V 7430 2600 50  0001 C CNN
+F 2 "Resistor_SMD:R_0805_2012Metric" V 7430 2600 50  0001 C CNN
 F 3 "~" H 7500 2600 50  0001 C CNN
 	1    7500 2600
@@
 F 0 "Y1" V 8004 1944 50  0000 L CNN
 F 1 "Crystal_GND24_Small" V 8095 1944 50  0000 L CNN
-F 2 "" H 8050 1800 50  0001 C CNN
+F 2 "Crystal:Crystal_SMD_3225-4Pin_3.2x2.5mm" H 8050 1800 50  0001 C CNN
 F 3 "~" H 8050 1800 50  0001 C CNN
 	1    8050 1800
@@
 F 0 "SW1" H 8350 1785 50  0000 C CNN
 F 1 "SW_Push" H 8350 1694 50  0000 C CNN
-F 2 "" H 8350 1700 50  0001 C CNN
+F 2 "random-keyboard-parts:SKQG-1155865" H 8350 1700 50  0001 C CNN
 F 3 "~" H 8350 1700 50  0001 C CNN
 	1    8350 1500
@@
 F 0 "R1" H 8659 1246 50  0000 L CNN
 F 1 "10k" H 8659 1155 50  0000 L CNN
-F 2 "" H 8600 1200 50  0001 C CNN
+F 2 "Resistor_SMD:R_0805_2012Metric" H 8600 1200 50  0001 C CNN
 F 3 "~" H 8600 1200 50  0001 C CNN
 	1    8600 1200
@@
 F 0 "R2" V 7743 2500 50  0000 C CNN
 F 1 "22" V 7834 2500 50  0000 C CNN
-F 2 "" V 7880 2500 50  0001 C CNN
+F 2 "Resistor_SMD:R_0805_2012Metric" V 7880 2500 50  0001 C CNN
 F 3 "~" H 7950 2500 50  0001 C CNN
 	1    7950 2500
@@
 F 0 "USB1" V 6687 1967 60  0000 C CNN
 F 1 "Molex-0548190589" V 6581 1967 60  0000 C CNN
-F 2 "" H 6150 2000 60  0001 C CNN
+F 2 "random-keyboard-parts:Molex-0548190589" H 6150 2000 60  0001 C CNN
 F 3 "" H 6150 2000 60  0001 C CNN
 	1    6150 2000
@@
 F 0 "F1" V 6675 1800 50  0000 C CNN
 F 1 "500mA" V 6766 1800 50  0000 C CNN
-F 2 "" H 6950 1600 50  0001 L CNN
+F 2 "Fuse:Fuse_1206_3216Metric" H 6950 1600 50  0001 L CNN
 F 3 "~" H 6900 1800 50  0001 C CNN
 	1    6900 1800
@@
 F 0 "MX1" H 6083 3273 60  0000 C CNN
 F 1 "MX-NoLED" H 6083 3199 20  0000 C CNN
-F 2 "" H 5425 3025 60  0001 C CNN
+F 2 "MX_Alps_Hybrid:MX-1U-NoLED" H 5425 3025 60  0001 C CNN
 F 3 "" H 5425 3025 60  0001 C CNN
 	1    6050 3050
@@
 F 0 "D1" V 5896 3230 50  0000 R CNN
 F 1 "D_Small" V 5805 3230 50  0000 R CNN
-F 2 "" V 5850 3300 50  0001 C CNN
+F 2 "Diode_SMD:D_SOD-123" V 5850 3300 50  0001 C CNN
 F 3 "~" V 5850 3300 50  0001 C CNN
 	1    5850 3300
@@
 F 0 "MX2" H 6633 3273 60  0000 C CNN
 F 1 "MX-NoLED" H 6633 3199 20  0000 C CNN
-F 2 "" H 5975 3025 60  0001 C CNN
+F 2 "MX_Alps_Hybrid:MX-1U-NoLED" H 5975 3025 60  0001 C CNN
 F 3 "" H 5975 3025 60  0001 C CNN
 	1    6600 3050
@@
 F 0 "D2" V 6446 3230 50  0000 R CNN
 F 1 "D_Small" V 6355 3230 50  0000 R CNN
-F 2 "" V 6400 3300 50  0001 C CNN
+F 2 "Diode_SMD:D_SOD-123" V 6400 3300 50  0001 C CNN
 F 3 "~" V 6400 3300 50  0001 C CNN
 	1    6400 3300
@@
 F 0 "MX3" H 6083 3873 60  0000 C CNN
 F 1 "MX-NoLED" H 6083 3799 20  0000 C CNN
-F 2 "" H 5425 3625 60  0001 C CNN
+F 2 "MX_Alps_Hybrid:MX-1U-NoLED" H 5425 3625 60  0001 C CNN
 F 3 "" H 5425 3625 60  0001 C CNN
 	1    6050 3650
@@
 F 0 "D3" V 5896 3830 50  0000 R CNN
 F 1 "D_Small" V 5805 3830 50  0000 R CNN
-F 2 "" V 5850 3900 50  0001 C CNN
+F 2 "Diode_SMD:D_SOD-123" V 5850 3900 50  0001 C CNN
 F 3 "~" V 5850 3900 50  0001 C CNN
 	1    5850 3900
@@
 F 0 "MX4" H 6633 3873 60  0000 C CNN
 F 1 "MX-NoLED" H 6633 3799 20  0000 C CNN
-F 2 "" H 5975 3625 60  0001 C CNN
+F 2 "MX_Alps_Hybrid:MX-1U-NoLED" H 5975 3625 60  0001 C CNN
 F 3 "" H 5975 3625 60  0001 C CNN
 	1    6600 3650
@@
 F 0 "D4" V 6446 3830 50  0000 R CNN
 F 1 "D_Small" V 6355 3830 50  0000 R CNN
-F 2 "" V 6400 3900 50  0001 C CNN
+F 2 "Diode_SMD:D_SOD-123" V 6400 3900 50  0001 C CNN
 F 3 "~" V 6400 3900 50  0001 C CNN
 	1    6400 3900

Commit message: finishing up pcb
Parts:
- MX1, MX2, MX3, MX4: footprint MX_Alps_Hybrid:MX-1U-NoLED -> MX_Alps_Hybrid:MX-1U
Connections:
- net COL0: now also U1.29 (PB5)
- net COL1: now also U1.28 (PB4)
- net ROW0: now also U1.27 (PD7)
- net ROW1: now also U1.30 (PB6)
Changed lines of the file:
@@
 	6450 2200 6550 2200
-$Comp
-L MX_Alps_Hybrid:MX-NoLED MX1
-U 1 1 6125CA13
-P 6050 3050
-F 0 "MX1" H 6083 3273 60  0000 C CNN
-F 1 "MX-NoLED" H 6083 3199 20  0000 C CNN
-F 2 "MX_Alps_Hybrid:MX-1U-NoLED" H 5425 3025 60  0001 C CNN
-F 3 "" H 5425 3025 60  0001 C CNN
-	1    6050 3050
-	1    0    0    -1
-$EndComp
 $Comp
 L Device:D_Small D1
@@
 	5850 3200 6000 3200
 $Comp
-L MX_Alps_Hybrid:MX-NoLED MX2
-U 1 1 61262832
-P 6600 3050
-F 0 "MX2" H 6633 3273 60  0000 C CNN
-F 1 "MX-NoLED" H 6633 3199 20  0000 C CNN
-F 2 "MX_Alps_Hybrid:MX-1U-NoLED" H 5975 3025 60  0001 C CNN
-F 3 "" H 5975 3025 60  0001 C CNN
-	1    6600 3050
-	1    0    0    -1
-$EndComp
-$Comp
 L Device:D_Small D2
 U 1 1 61262838
@@
 	6400 3200 6550 3200
 $Comp
-L MX_Alps_Hybrid:MX-NoLED MX3
-U 1 1 61263ED7
-P 6050 3650
-F 0 "MX3" H 6083 3873 60  0000 C CNN
-F 1 "MX-NoLED" H 6083 3799 20  0000 C CNN
-F 2 "MX_Alps_Hybrid:MX-1U-NoLED" H 5425 3625 60  0001 C CNN
-F 3 "" H 5425 3625 60  0001 C CNN
-	1    6050 3650
-	1    0    0    -1
-$EndComp
-$Comp
 L Device:D_Small D3
 U 1 1 61263EDD
@@
 Wire Wire Line
 	5850 3800 6000 3800
-$Comp
-L MX_Alps_Hybrid:MX-NoLED MX4
-U 1 1 61265E05
-P 6600 3650
-F 0 "MX4" H 6633 3873 60  0000 C CNN
-F 1 "MX-NoLED" H 6633 3799 20  0000 C CNN
-F 2 "MX_Alps_Hybrid:MX-1U-NoLED" H 5975 3625 60  0001 C CNN
-F 3 "" H 5975 3625 60  0001 C CNN
-	1    6600 3650
-	1    0    0    -1
-$EndComp
 $Comp
 L Device:D_Small D4
@@
 Wire Wire Line
 	5850 4000 5650 4000
-Wire Wire Line
-	6200 3600 6200 3000
-Connection ~ 6200 3000
-Wire Wire Line
-	6200 3000 6200 2700
-Wire Wire Line
-	6750 3600 6750 3000
-Connection ~ 6750 3000
-Wire Wire Line
-	6750 3000 6750 2700
 Text GLabel 6750 2700 1    50   Input ~ 0
 COL1
@@
 Text GLabel 5650 4000 0    50   Input ~ 0
 ROW1
+Text GLabel 9900 1900 2    50   Input ~ 0
+COL1
+Text GLabel 9900 2000 2    50   Input ~ 0
+COL0
+Text GLabel 9900 2100 2    50   Input ~ 0
+ROW1
+Text GLabel 9900 3400 2    50   Input ~ 0
+ROW0
+$Comp
+L MX_Alps_Hybrid:MX-NoLED MX3
+U 1 1 61263ED7
+P 6050 3650
+F 0 "MX3" H 6083 3873 60  0000 C CNN
+F 1 "MX-NoLED" H 6083 3799 20  0000 C CNN
+F 2 "MX_Alps_Hybrid:MX-1U" H 5425 3625 60  0001 C CNN
+F 3 "" H 5425 3625 60  0001 C CNN
+	1    6050 3650
+	1    0    0    -1
+$EndComp
+$Comp
+L MX_Alps_Hybrid:MX-NoLED MX4
+U 1 1 61265E05
+P 6600 3650
+F 0 "MX4" H 6633 3873 60  0000 C CNN
+F 1 "MX-NoLED" H 6633 3799 20  0000 C CNN
+F 2 "MX_Alps_Hybrid:MX-1U" H 5975 3625 60  0001 C CNN
+F 3 "" H 5975 3625 60  0001 C CNN
+	1    6600 3650
+	1    0    0    -1
+$EndComp
+Wire Wire Line
+	6750 3000 6750 2700
+Wire Wire Line
+	6750 3600 6750 3000
+Connection ~ 6750 3000
+$Comp
+L MX_Alps_Hybrid:MX-NoLED MX2
+U 1 1 61262832
+P 6600 3050
+F 0 "MX2" H 6633 3273 60  0000 C CNN
+F 1 "MX-NoLED" H 6633 3199 20  0000 C CNN
+F 2 "MX_Alps_Hybrid:MX-1U" H 5975 3025 60  0001 C CNN
+F 3 "" H 5975 3025 60  0001 C CNN
+	1    6600 3050
+	1    0    0    -1
+$EndComp
+Connection ~ 6200 3000
+Wire Wire Line
+	6200 3000 6200 2700
+Wire Wire Line
+	6200 3600 6200 3000
+$Comp
+L MX_Alps_Hybrid:MX-NoLED MX1
+U 1 1 6125CA13
+P 6050 3050
+F 0 "MX1" H 6083 3273 60  0000 C CNN
+F 1 "MX-NoLED" H 6083 3199 20  0000 C CNN
+F 2 "MX_Alps_Hybrid:MX-1U" H 5425 3025 60  0001 C CNN
+F 3 "" H 5425 3025 60  0001 C CNN
+	1    6050 3050
+	1    0    0    -1
+$EndComp
 $EndSCHEMATC
