File: ai03-pcb-guide/ai03-pcb-guide.kicad_pcb (KiCad board)
At the start: 2 copper layers, 24 parts, among them SW1 SW_Push, U1 ATmega32U4-A, Y1 Crystal_GND24_Small

Commit message: finishing up pcb
Parts:
- D1, D2, D3, D4, USB1: moved to B.Cu
- MX1, MX2, MX3, MX4: footprint MX_Alps_Hybrid:MX-1U-NoLED -> MX_Alps_Hybrid:MX-1U
- moved D4 73.0 mm to (129.4, 54.0)
- moved D1 73.0 mm to (110.3, 34.9)
- moved D2 73.0 mm to (129.4, 34.9)
- moved D3 73.0 mm to (110.3, 53.9)
- moved MX1 72.2 mm to (101.6, 34.9)
- moved MX3 72.2 mm to (101.6, 54.0)
- moved MX4 72.2 mm to (120.7, 54.0)
- moved MX2 72.2 mm to (120.7, 34.9)
- moved C7 8.05 mm to (69.8, 47.8), turned to 270 degrees
- moved R2 5.32 mm to (64.9, 36.9)
- moved R3 5.32 mm to (62.6, 36.9)
- moved SW1 4.43 mm to (62.0, 55.0)
- moved F1 3.76 mm to (58.7, 38.7), turned to 90 degrees
- moved USB1 1.49 mm to (64.3, 27.0)
- moved R1 1.03 mm to (68.3, 35.8), turned to 270 degrees
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Connections:
- U1 pad 27: Net-(U1-Pad27) -> ROW0
- U1 pad 28: Net-(U1-Pad28) -> COL1
- U1 pad 29: Net-(U1-Pad29) -> COL0
- U1 pad 30: Net-(U1-Pad30) -> ROW1
Routing:
- net GND: track 0.00 -> 145.5 mm
- net +5V: track 0.00 -> 101.3 mm, vias 0 -> 6
- net ROW1: track 0.00 -> 55.0 mm
- net COL1: track 0.00 -> 53.2 mm
- net ROW0: track 0.00 -> 46.7 mm
- net COL0: track 0.00 -> 33.9 mm
- net Net-(R1-Pad2): track 0.00 -> 30.1 mm, vias 0 -> 2
- net Net-(R3-Pad1): track 0.00 -> 17.3 mm
- net Net-(R2-Pad1): track 0.00 -> 16.1 mm
- net Net-(C2-Pad1): track 0.00 -> 12.5 mm
- net Net-(C1-Pad1): track 0.00 -> 9.19 mm
- net Net-(D4-Pad2): track 0.00 -> 9.08 mm
- net Net-(D2-Pad2): track 0.00 -> 9.00 mm
- net Net-(D1-Pad2): track 0.00 -> 8.28 mm
- net Net-(D3-Pad2): track 0.00 -> 7.98 mm
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- added copper zone on B.Cu, net GND
Other:
- board outline added: 77 x 38.1 mm
- net class Default: trace_width 0.25 -> 0.254
- net class power added: clearance 0.2, trace_width 0.381, via_dia 0.8, via_drill 0.4
- rule trace_min: 0.2 -> 0.000178
- board text added: "Nhan Ha"

Commit message: finalizing and fixing up routes
Parts:
- moved R3 0.14 mm to (62.7, 36.9)
Routing:
- net Net-(R4-Pad2): track 0.00 -> 3.76 mm
- net +5V: track 101.3 -> 102.9 mm
- net Net-(D2-Pad2): track 9.00 -> 7.59 mm
- net VCC: track 7.46 -> 8.41 mm
- net ROW1: track 55.0 -> 54.3 mm
- net ROW0: track 46.7 -> 47.4 mm
- net Net-(D1-Pad2): track 8.28 -> 7.69 mm
Other:
- board size 77 x 38.1 mm -> 79.4 x 38.1 mm
